File: rj45-kicad/rj45.kicad_sch (KiCad schematic)
At the start: 46 parts

Commit message: Schema electrica
Other:
- title: (none) -> RJ-45 Tester (by Trifan Bogdan-Cristian)
Changed lines of the file:
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@@
 (kicad_sch (version 20211123) (generator eeschema)
   (paper "A4")
+  (title_block
+    (title "RJ-45 Tester (by Trifan Bogdan-Cristian)")
+  )
   (junction (at 113.03 86.36) (diameter 0) (color 0 0 0 0)
   )
